File: kicad/alleycat.kicad_sch (KiCad schematic)
At the start: 94 parts, among them J1 Conn_01x04_Female, J2 USB_C_Receptacle_USB2.0, J3 Conn_01x04_Male, SW1 RotaryEncoder_Switch, SW2 SW_Push, U1 E73-2G4M08S1C, U2 MCP73831-2-OT

Commit message: fot
Parts:
- MX1, MX10, MX11, MX12, MX13, MX14, MX15, MX16, MX17, MX18, MX19, MX2, MX20, MX21, MX22, MX23, MX24, MX25, MX26, MX27, MX28, MX29, MX3, MX30, MX31, MX32, MX33, MX34, MX35, MX37, MX4, MX5, MX6, MX7, MX8, MX9: footprint MX_Only:MXOnly-1U-NoLED -> MX:MXOnly-1U-Hotswap
- MX36: footprint MX_Only:MXOnly-1U-NoLED -> MX:MXOnly-2U-Hotswap

Commit message: wicked usb
Parts:
- J2: footprint (none) -> MX:TYPE-C-31-M-12
Changed lines of the file:
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@@
     (property "Reference" "J2" (id 0) (at 216.535 15.24 0))
     (property "Value" "USB_C_Receptacle_USB2.0" (id 1) (at 216.535 17.78 0))
-    (property "Footprint" "" (id 2) (at 220.345 38.735 0)
+    (property "Footprint" "MX:TYPE-C-31-M-12" (id 2) (at 220.345 38.735 0)
       (effects (font (size 1.27 1.27)) hide)
     )
@@
     )
     (path "/34a9dc99-5ad8-4b25-988b-4ecfd1ccb6d1"
-      (reference "J2") (unit 1) (value "USB_C_Receptacle_USB2.0") (footprint "")
+      (reference "J2") (unit 1) (value "USB_C_Receptacle_USB2.0") (footprint "MX:TYPE-C-31-M-12")
     )
     (path "/9bd6d535-7d29-4770-92a1-5b2eb4caf31e"
