File: kicad/alleycat.kicad_sch (KiCad schematic)
At the start: 94 parts, among them J1 Conn_01x04_Female, J2 USB_C_Receptacle_USB2.0, J3 Conn_01x04_Male, SW1 RotaryEncoder_Switch, SW2 SW_Push

Commit message: battery management
Parts:
- added C1: 10uf, symbol Device:C_Small
- added C2: 100nf, symbol Device:C_Polarized_Small
- added C3: 100nf, symbol Device:C_Small
- added D44, D45: LED, symbol Device:LED_Small
- added JP1: THERM, symbol Jumper:SolderJumper_2_Open
- added R1, R4: 2.7k, symbol Device:R_Small
- added R5: 1.8k, symbol Device:R_Small
- added R6: 3.3k, symbol Device:R_Small
- added R7: 22k, symbol Device:R_Small
- added R8: 100, symbol Device:R_Small
- added R9: 1k, symbol Device:R_Small
- added U2: DW01A, Package_TO_SOT_SMD:SOT-23-6, symbol marbastlib-various:DW01A
- added U3: FS8205, Package_TO_SOT_SMD:SOT-23-6, symbol marbastlib-various:FS8205
- gave numbers to parts that had none: 1
Connections:
- net +5V: now also U1.4 (VCC), U1.8 (CE), C1.1, C2.1, D44.2 (A), D45.2 (A), R6.1
- net GND: now also U1.3 (GND), C1.2, C2.2, JP1.1 (A), R5.2, R7.2, R9.2, U3.3 (S2)
- net d+: no longer J2.A6 (D+), J2.B6 (D+), U?.1 (IO1)
- net d-: no longer J2.A7 (D-), J2.B7 (D-), U?.4 (IO3)
- net vbus: no longer F?.1, J2.A4 (VBUS), J2.A9 (VBUS), J2.B4 (VBUS), J2.B9 (VBUS)
- net at D7.2 (A), S1.1 (A): no longer D35.2 (A), S1.7 (COM)
- net at U1.1 (TEMP): now also JP1.2 (B), R6.2, R7.1
- net at U1.2 (PROG): now also R5.1
- net BAT+: now reaches U1.5 (BAT)
- net BAT+: now also R8.1
- net at U1.6 (STDBY): now also R4.1
- net at U1.7 (CHRG): now also R1.1
- new net: C3.1, R8.2, U2.5 (VDD)
- new net: U2.1 (OD), U3.6 (G1)
- new net: R9.1, U2.2 (CSI)
- new net: U2.3 (OC), U3.4 (G2)
- new net: D35.2 (A), S1.7 (COM)
- new net: D44.1 (K), R1.2
- new net: D45.1 (K), R4.2
- new net BAT-: C3.2, U2.6 (VSS), U3.1 (S1)
- new net D+: J2.A6 (D+), J2.B6 (D+), U?.1 (IO1)
- new net D-: J2.A7 (D-), J2.B7 (D-), U?.4 (IO3)
- new net VBUS: F?.1, J2.A4 (VBUS), J2.A9 (VBUS), J2.B4 (VBUS), J2.B9 (VBUS)
- no-connect marks 14 -> 17
Other:
- moved on the sheet: D16, D35, D36, D7, D8, D9, F?, J1, J2, R2, R3, S1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

Commit message: wicked voltage regulator
Parts:
- added C4, C5: 4.7uf, symbol Device:C_Small
- added C6, C7: 1uf, symbol Device:C_Small
- added C8: 100nf, symbol Device:C_Small
- added R10: 806k, symbol Device:R_Small
- added R11: 2M, symbol Device:R_Small
- added U6: XC6206PxxxMR, Package_TO_SOT_SMD:SOT-23, symbol Regulator_Linear:XC6206PxxxMR
- gave numbers to parts that had none: 4
- renumbered D13 to D10, D14 to D11, D15 to D12, D17 to D13, D18 to D14, D19 to D15, D20 to D16, D21 to D17, D22 to D18, D23 to D19, D24 to D20, D25 to D21, D26 to D22, D27 to D23, D28 to D24, D29 to D25, D30 to D26, D31 to D27, D32 to D28, D33 to D29, D34 to D30, D37 to D31, D38 to D32, D39 to D33, D40 to D34, D41 to D35, D42 to D36, D43 to D37, D44 to D38, D45 to D39, D7 to D40, D8 to D41, D9 to D42, D16 to D44, D35 to D45, D36 to D46, D10 to D7, D11 to D8, D12 to D9, J3 to J1, J1 to J3, R4 to R2, R5 to R3, R6 to R4, R7 to R5, R2 to R6, R3 to R7, SW2 to SW1, SW1 to SW2, U1 to U2, U2 to U3, U3 to U4
Connections:
- net +3.3V: now also C7.1, C8.1, U6.2 (VO)
- net BAT+: now also C4.1, C5.1, C6.1, R10.2, U6.3 (VI)
- net GND: now also C4.2, C5.2, C6.2, C7.2, C8.2, R11.1, U6.1 (GND)
- net VSENSE: now reaches U1.11 (P0.31)
- net VSENSE: now also R10.1, R11.2
Other:
- note added: "rug"

Commit message: uhh uhhh uhhh uhh uhhh uhhh uhhh uuhhh uhhh uhh uhh uhhhu hh uhh footprints
Parts:
- C1, C2, C3, C4, C5, C6, C7, C8: footprint (none) -> Capacitor_SMD:C_0805_2012Metric
- D38, D39: footprint (none) -> LED_SMD:LED_0805_2012Metric
- D43: footprint (none) -> MX:SOD-323
- F1: footprint (none) -> Fuse:Fuse_1206_3216Metric
- JP1: footprint (none) -> Jumper:SolderJumper-2_P1.3mm_Open_TrianglePad1.0x1.5mm
- L1: footprint (none) -> Capacitor_SMD:C_0402_1005Metric
- R1, R10, R11, R2, R3, R4, R5, R8, R9: footprint (none) -> Resistor_SMD:R_0805_2012Metric

Commit message: pcb edit pog pog pog
Connections:
- net +5V: now also J1.2 (Pin_2)
- net vbus: no longer J1.2 (Pin_2)
Changed lines of the file:
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@@
-    )
-  )
-  (global_label "vbus" (shape input) (at 45.72 266.7 270) (fields_autoplaced)
-    (effects (font (size 1.27 1.27)) (justify right))
-    (property "Intersheet References" "${INTERSHEET_REFS}" (id 0) (at 45.6406 273.4069 90)
-      (effects (font (size 1.27 1.27)) (justify right) hide)
     )
   )
@@
     (pin "1")
     (pin "2")
+  )
+  (symbol (lib_id "power:+5V") (at 45.72 266.7 180) (unit 1)
+    (in_bom yes) (on_board yes) (fields_autoplaced)
+    (property "Reference" "#PWR?" (id 0) (at 45.72 262.89 0)
+      (effects (font (size 1.27 1.27)) hide)
+    )
+    (property "Value" "+5V" (id 1) (at 45.72 271.78 0))
+    (property "Footprint" "" (id 2) (at 45.72 266.7 0)
+      (effects (font (size 1.27 1.27)) hide)
+    )
+    (property "Datasheet" "" (id 3) (at 45.72 266.7 0)
+      (effects (font (size 1.27 1.27)) hide)
+    )
+    (pin "1")
   )
   (symbol (lib_id "Device:R_Small") (at 163.83 140.97 0) (unit 1)
@@
       (reference "#PWR027") (unit 1) (value "+3.3V") (footprint "")
     )
+    (path "/cbf94107-943d-4133-8ad6-7916fb9ebd37"
+      (reference "#PWR?") (unit 1) (value "+5V") (footprint "")
+    )
     (path "/e80f4818-6806-41f2-b9c3-d610345fa90c"

Commit message: changed io protector pin so it isnt stupid
Connections:
- net D-: now also U5.3 (IO2); no longer U5.4 (IO3)
Changed lines of the file:
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@@
   (no_connect (at 255.27 143.51))
   (no_connect (at 255.27 128.27))
-  (no_connect (at 275.59 44.45))
   (no_connect (at 250.19 49.53))
+  (no_connect (at 275.59 49.53))
   (no_connect (at -15.875 -17.145))
   (no_connect (at -15.875 -19.685))
@@
     (stroke (width 0) (type default) (color 0 0 0 0))
   )
-  (wire (pts (xy 275.59 49.53) (xy 276.86 49.53))
+  (wire (pts (xy 275.59 44.45) (xy 276.86 44.45))
     (stroke (width 0) (type default) (color 0 0 0 0))
   )
@@
     )
   )
-  (global_label "D-" (shape input) (at 276.86 49.53 0) (fields_autoplaced)
+  (global_label "D-" (shape input) (at 276.86 44.45 0) (fields_autoplaced)
     (effects (font (size 1.27 1.27)) (justify left))
-    (property "Intersheet References" "${INTERSHEET_REFS}" (id 0) (at 282.1155 49.4506 0)
+    (property "Intersheet References" "${INTERSHEET_REFS}" (id 0) (at 282.1155 44.3706 0)
       (effects (font (size 1.27 1.27)) (justify left) hide)
     )

Commit message: a
Parts:
- U2: footprint Package_SO:SOP-8-1EP_4.57x4.57mm_P1.27mm_EP4.57x4.45mm -> Package_SO:SOP-8_3.76x4.96mm_P1.27mm
Changed lines of the file:
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@@
     (property "Reference" "U2" (id 0) (at 180.975 116.84 0))
     (property "Value" "TP4056" (id 1) (at 180.975 119.38 0))
-    (property "Footprint" "Package_SO:SOP-8-1EP_4.57x4.57mm_P1.27mm_EP4.57x4.45mm" (id 2) (at 180.34 116.84 0)
+    (property "Footprint" "Package_SO:SOP-8_3.76x4.96mm_P1.27mm" (id 2) (at 180.34 116.84 0)
       (effects (font (size 1.27 1.27)) hide)
     )
@@
   (symbol (lib_id "power:+5V") (at 45.72 266.7 180) (unit 1)
     (in_bom yes) (on_board yes) (fields_autoplaced)
-    (property "Reference" "#PWR?" (id 0) (at 45.72 262.89 0)
+    (property "Reference" "#PWR0101" (id 0) (at 45.72 262.89 0)
       (effects (font (size 1.27 1.27)) hide)
     )
@@
     )
     (path "/cbf94107-943d-4133-8ad6-7916fb9ebd37"
-      (reference "#PWR?") (unit 1) (value "+5V") (footprint "")
+      (reference "#PWR0101") (unit 1) (value "+5V") (footprint "")
     )
     (path "/e80f4818-6806-41f2-b9c3-d610345fa90c"
@@
     )
     (path "/80ece84b-18d0-4126-af64-908a1c7d4ea8"
-      (reference "U2") (unit 1) (value "TP4056") (footprint "Package_SO:SOP-8-1EP_4.57x4.57mm_P1.27mm_EP4.57x4.45mm")
+      (reference "U2") (unit 1) (value "TP4056") (footprint "Package_SO:SOP-8_3.76x4.96mm_P1.27mm")
     )
     (path "/3e90c7eb-e997-4415-900d-3f8c14c03069"
