File: kicad/alleycat.kicad_pcb (KiCad board)
At the start: 2 copper layers, 144 x 131 mm, 84 parts, among them J1 Conn_01x04_Female, SW1 RotaryEncoder_Switch, U1 E73-2G4M08S1C

Commit message: wicked
Parts:
- MX1, MX10, MX11, MX12, MX13, MX14, MX15, MX16, MX17, MX18, MX19, MX2, MX20, MX21, MX22, MX23, MX24, MX25, MX26, MX27, MX28, MX29, MX3, MX30, MX31, MX32, MX33, MX34, MX35, MX36, MX37, MX4, MX5, MX6, MX7, MX8, MX9: footprint MX_Only:MXOnly-1U-NoLED -> MX:MX-NoLED
- moved MX2 171.0 mm to (159.2, 166.5)
- moved MX1 157.7 mm to (185.2, 73.5)
- moved MX28 124.7 mm to (131.2, 179.5)
Other:
- board size 144 x 131 mm -> 134 x 128 mm

Commit message: a
Parts:
- added C1: 10uf, Capacitor_SMD:C_0805_2012Metric, B.Cu at (204.0, 99.0)
- added C2: 100nf, Capacitor_SMD:C_0805_2012Metric, B.Cu at (263.4, 38.5)
- added C3: 100nf, Capacitor_SMD:C_0805_2012Metric, B.Cu at (106.5, 158.1)
- added C4: 4.7uf, Capacitor_SMD:C_0805_2012Metric, B.Cu at (157.8, 142.8)
- added C5: 4.7uf, Capacitor_SMD:C_0805_2012Metric, B.Cu at (72.2, 153.4)
- added C6: 1uf, Capacitor_SMD:C_0805_2012Metric, B.Cu at (243.2, 58.7)
- added C7: 1uf, Capacitor_SMD:C_0805_2012Metric, B.Cu at (198.2, 102.3)
- added C8: 100nf, Capacitor_SMD:C_0805_2012Metric, B.Cu at (257.6, 45.2)
- added D44: D_Small, Diode_SMD:D_SOD-123, B.Cu at (178.7, 119.5)
- added D45: D_Small, Diode_SMD:D_SOD-123, B.Cu at (90.0, 156.7)
- added D46: D_Small, Diode_SMD:D_SOD-123, B.Cu at (198.9, 79.1)
- added F1: Polyfuse_Small, Fuse:Fuse_1206_3216Metric, B.Cu at (101.5, 158.2)
- added J2: USB_C_Receptacle_USB2.0, MX:TYPE-C-31-M-12, B.Cu at (98.7, 140.9)
- added JP1: THERM, Jumper:SolderJumper-2_P1.3mm_Open_TrianglePad1.0x1.5mm, B.Cu at (198.2, 105.6)
- added L1: L, Capacitor_SMD:C_0402_1005Metric, B.Cu at (94.8, 153.1)
- added R1: 2.7k, Resistor_SMD:R_0805_2012Metric, B.Cu at (183.8, 119.3)
- added R10: 806k, Resistor_SMD:R_0805_2012Metric, B.Cu at (243.2, 61.7)
- added R11: 2M, Resistor_SMD:R_0805_2012Metric, B.Cu at (209.7, 95.3)
- added R2: 2.7k, Resistor_SMD:R_0805_2012Metric, B.Cu at (202.7, 102.3)
- added R3: 1.8k, Resistor_SMD:R_0805_2012Metric, B.Cu at (221.2, 82.2)
- added R4: 3.3k, Resistor_SMD:R_0805_2012Metric, B.Cu at (163.6, 139.5)
- added R5: 22k, Resistor_SMD:R_0805_2012Metric, B.Cu at (227.0, 78.9)
- added R6: 5.1k, Resistor_SMD:R_0805_2012Metric, B.Cu at (257.6, 48.2)
- added R7: 5.1k, Resistor_SMD:R_0805_2012Metric, B.Cu at (263.4, 41.5)
- added R8: 100, Resistor_SMD:R_0805_2012Metric, B.Cu at (237.5, 65.4)
- added R9: 1k, Resistor_SMD:R_0805_2012Metric, B.Cu at (237.5, 68.3)
- added SW2: RotaryEncoder_Switch, Keebio-Parts:RotaryEncoder_Alps_EC11E-Switch_Vertical_H20mm, B.Cu at (84.3, 147.4)
- added U2: TP4056, Package_SO:MSOP-8-1EP_3x3mm_P0.65mm_EP1.95x2.15mm, B.Cu at (81.2, 74.2)
- added U3: DW01A, Package_TO_SOT_SMD:SOT-23-6, B.Cu at (178.4, 123.4)
- added U4: FS8205, Package_TO_SOT_SMD:SOT-23-6, B.Cu at (215.8, 86.3)
- added U5: SRV05-4, marbastlib-various:SOT-23-6-routable, B.Cu at (112.3, 145.1)
- added U6: XC6206PxxxMR, Package_TO_SOT_SMD:SOT-23, B.Cu at (112.6, 155.4)
- D1, D10, D11, D12, D13, D14, D15, D16, D17, D18, D19, D2, D20, D21, D22, D23, D24, D25, D26, D27, D28, D29, D3, D30, D31, D32, D33, D34, D35, D36, D37, D4, D40, D41, D42, D5, D6, D7, D8, D9: moved to B.Cu
- D38, D39: value D_Small -> LED; footprint Diode_SMD:D_SOD-123 -> LED_SMD:LED_0805_2012Metric; moved to B.Cu
- D43: value D_Small -> D_TVS; footprint Diode_SMD:D_SOD-123 -> MX:SOD-323; moved to B.Cu
- J1: value Conn_01x04_Female -> Conn_01x04_Male
- MX1, MX10, MX11, MX12, MX13, MX14, MX15, MX16, MX17, MX18, MX19, MX2, MX20, MX21, MX22, MX23, MX24, MX25, MX26, MX27, MX28, MX29, MX3, MX30, MX31, MX32, MX33, MX34, MX35, MX37, MX4, MX5, MX6, MX7, MX8, MX9: footprint MX:MX-NoLED -> MX:MXOnly-1U-Hotswap
- MX36: footprint MX:MX-NoLED -> MX:MXOnly-2U-Hotswap
- SW1: value RotaryEncoder_Switch -> SW_Push; footprint Keebio-Parts:RotaryEncoder_Alps_EC11E-Switch_Vertical_H20mm -> Keebio-Parts:SW_SPST_TL3342; moved to B.Cu
- U1: value E73-2G4M08S1C -> nRF52840_holyiot_18010; footprint E73-2G4M08S1C:E73-2G4M08S1C -> marbastlib-various:nRF52840_holyiot_18010; moved to B.Cu
- moved MX32 301.6 mm to (57.6, 78.7)
- moved MX3 280.9 mm to (57.6, 98.9)
- moved MX11 266.2 mm to (118.2, 125.4)
- moved MX18 235.4 mm to (98.0, 127.2)
- moved MX30 223.0 mm to (118.2, 85.0)
- moved MX5 220.3 mm to (77.8, 127.2)
- moved MX20 213.6 mm to (57.6, 119.1)
- moved MX12 213.0 mm to (57.6, 139.3)
- moved MX9 209.2 mm to (118.2, 145.6)
- moved MX36 207.8 mm to (67.2, 57.8)
- moved MX31 202.6 mm to (118.2, 105.2)
- moved MX29 199.2 mm to (177.6, 44.6)
- moved MX37 181.1 mm to (77.8, 86.8)
- moved D21 180.4 mm to (84.3, 156.7), turned to 180 degrees
- moved D37 180.2 mm to (90.4, 72.8), turned to 180 degrees
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Connections:
- net circle_X renamed sda
- D10 pad 1: row_5 -> row_2
- D11 pad 1: row_4 -> row_1
- D12 pad 1: row_3 -> row_0
- D13 pad 1: row_2 -> row_5
- D14 pad 1: row_1 -> row_4
- D15 pad 1: row_0 -> row_3
- D16 pad 1: row_0 -> row_2
- D17 pad 1: row_5 -> row_1
- D18 pad 1: row_4 -> row_0
- D19 pad 1: row_3 -> row_5
- D20 pad 1: row_2 -> row_4
- D21 pad 1: row_1 -> row_3
- D22 pad 1: row_0 -> row_2
- D23 pad 1: row_5 -> row_1
- D24 pad 1: row_4 -> row_0
- D25 pad 1: row_3 -> row_5
- D26 pad 1: row_2 -> row_4
- D27 pad 1: row_1 -> row_3
- D28 pad 1: row_0 -> row_2
- D29 pad 1: row_5 -> row_1
- D30 pad 1: row_4 -> row_0
- D31 pad 1: row_3 -> row_5
- D32 pad 1: row_2 -> row_4
- D33 pad 1: row_1 -> row_3
- D34 pad 1: row_0 -> row_2
- D35 pad 1: row_4 -> row_1
- D36 pad 1: row_3 -> row_0
- D38 pad 1: row_4 -> Net-(D38-Pad1)
- D38 pad 2: Net-(D38-Pad2) -> +5V
- D39 pad 1: row_3 -> Net-(D39-Pad1)
- D39 pad 2: Net-(D39-Pad2) -> +5V
- D40 pad 1: row_2 -> row_0
- D42 pad 1: row_0 -> row_2
- D7 pad 1: row_0 -> row_5
- D7 pad 2: Net-(D35-Pad2) -> Net-(D7-Pad2)
- D8 pad 1: row_1 -> row_4
- D9 pad 1: row_2 -> row_3
- J1 pad 2: circle_Y -> +5V
- J1 pad 3: +5V -> scl
- MX10 pad 2: Net-(D13-Pad2) -> Net-(D10-Pad2)
- MX11 pad 2: Net-(D14-Pad2) -> Net-(D11-Pad2)
- MX12 pad 2: Net-(D15-Pad2) -> Net-(D12-Pad2)
- MX13 pad 2: Net-(D17-Pad2) -> Net-(D13-Pad2)
- MX14 pad 2: Net-(D18-Pad2) -> Net-(D14-Pad2)
- MX15 pad 2: Net-(D19-Pad2) -> Net-(D15-Pad2)
- MX16 pad 2: Net-(D20-Pad2) -> Net-(D16-Pad2)
- MX17 pad 2: Net-(D21-Pad2) -> Net-(D17-Pad2)
- MX18 pad 2: Net-(D22-Pad2) -> Net-(D18-Pad2)
- MX19 pad 2: Net-(D23-Pad2) -> Net-(D19-Pad2)
- MX20 pad 2: Net-(D24-Pad2) -> Net-(D20-Pad2)
- MX21 pad 2: Net-(D25-Pad2) -> Net-(D21-Pad2)
- MX22 pad 2: Net-(D26-Pad2) -> Net-(D22-Pad2)
- MX23 pad 2: Net-(D27-Pad2) -> Net-(D23-Pad2)
- MX24 pad 2: Net-(D28-Pad2) -> Net-(D24-Pad2)
- MX25 pad 2: Net-(D29-Pad2) -> Net-(D25-Pad2)
- MX26 pad 2: Net-(D30-Pad2) -> Net-(D26-Pad2)
- MX27 pad 2: Net-(D31-Pad2) -> Net-(D27-Pad2)
- MX28 pad 2: Net-(D32-Pad2) -> Net-(D28-Pad2)
- MX29 pad 2: Net-(D33-Pad2) -> Net-(D29-Pad2)
- MX30 pad 2: Net-(D34-Pad2) -> Net-(D30-Pad2)
- MX31 pad 2: Net-(D37-Pad2) -> Net-(D31-Pad2)
- MX32 pad 2: Net-(D38-Pad2) -> Net-(D32-Pad2)
- MX33 pad 2: Net-(D39-Pad2) -> Net-(D33-Pad2)
- MX34 pad 2: Net-(D40-Pad2) -> Net-(D34-Pad2)
- MX35 pad 2: Net-(D41-Pad2) -> Net-(D35-Pad2)
- MX36 pad 2: Net-(D42-Pad2) -> Net-(D36-Pad2)
- MX37 pad 2: Net-(D43-Pad2) -> Net-(D37-Pad2)
- MX7 pad 2: Net-(D10-Pad2) -> Net-(D7-Pad2)
- MX8 pad 2: Net-(D11-Pad2) -> Net-(D8-Pad2)
- MX9 pad 2: Net-(D12-Pad2) -> Net-(D9-Pad2)
- S1 pad 1: Net-(D35-Pad2) -> Net-(D40-Pad2)
- S1 pad 4: Net-(D8-Pad2) -> Net-(D41-Pad2)
- S1 pad 6: Net-(D9-Pad2) -> Net-(D42-Pad2)
- S1 pad 7: Net-(D35-Pad2) -> Net-(D45-Pad2)
- S1 pad 9: Net-(D36-Pad2) -> Net-(D46-Pad2)
- U1 pad 11: unconnected-(U1-Pad11) -> VSENSE
- U1 pad 14: unconnected-(U1-Pad14) -> +3.3V
- U1 pad 21: unconnected-(U1-Pad21) -> reset
- U1 pad 22: unconnected-(U1-Pad22) -> vbus
- U1 pad 23: unconnected-(U1-Pad23) -> d-
- U1 pad 24: unconnected-(U1-Pad24) -> d+
- U1 pad 31: unconnected-(U1-Pad31) -> swdclk
- U1 pad 32: unconnected-(U1-Pad32) -> swdio
Routing:
- added copper zone on B.Cu, net GND
Other:
- board size 134 x 128 mm -> 225 x 136 mm
