File: kicad/right/alleycat_right.kicad_pcb (KiCad board)
At the start: 2 copper layers, 134 x 128 mm, 85 parts, among them J1 Conn_01x04_Female, SW1 RotaryEncoder_Switch, U1 E73-2G4M08S1C, U2 MCP73831-2-OT

Commit message: ANY ALIGNERS?
Parts:
- MX1, MX10, MX11, MX12, MX13, MX14, MX15, MX16, MX17, MX18, MX19, MX2, MX20, MX21, MX22, MX23, MX24, MX25, MX26, MX27, MX28, MX29, MX3, MX30, MX31, MX32, MX33, MX34, MX35, MX36, MX37, MX4, MX5, MX6, MX7, MX8, MX9: value MX-NoLED -> 1U; footprint MX:MX-NoLED -> MX:MXOnly-1U-Hotswap
- moved MX29 326.4 mm to (56.0, 99.0)
- moved MX32 319.6 mm to (37.0, 42.0)
- moved MX30 293.5 mm to (54.5, 120.6), turned to 10 degrees
- moved MX27 281.3 mm to (56.0, 61.0)
- moved MX31 280.7 mm to (37.0, 23.0)
- moved MX11 265.9 mm to (113.1, 99.0)
- moved MX34 262.2 mm to (37.0, 80.0)
- moved MX36 258.2 mm to (26.0, 127.0)
- moved MX37 256.7 mm to (18.0, 23.0)
- moved MX26 243.2 mm to (56.0, 42.0)
- moved MX19 241.4 mm to (75.0, 23.0)
- moved MX18 235.9 mm to (94.0, 118.0)
- moved MX21 209.4 mm to (75.0, 61.0)
- moved MX10 204.3 mm to (113.1, 80.0)
- moved MX9 204.2 mm to (113.1, 61.0)
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
Commit message: wicked usb
Parts:
- added J2: USB_C_Receptacle_USB2.0, MX:TYPE-C-31-M-12, F.Cu at (174.0, 17.0)
- MX1, MX10, MX11, MX12, MX13, MX14, MX15, MX16, MX17, MX18, MX19, MX2, MX20, MX21, MX22, MX23, MX24, MX25, MX26, MX27, MX28, MX29, MX3, MX30, MX31, MX32, MX33, MX34, MX35, MX36, MX37, MX4, MX5, MX6, MX7, MX8, MX9: value 1U -> MX-NoLED

Commit message: uhh uhhh uhhh uhh uhhh uhhh uhhh uuhhh uhhh uhh uhh uhhhu hh uhh footprints
Parts:
- added C1: 10uf, Capacitor_SMD:C_0805_2012Metric, F.Cu at (174.0, 87.0)
- added C2: 100nf, Capacitor_SMD:C_0805_2012Metric, F.Cu at (185.0, 76.2)
- added C3: 100nf, Capacitor_SMD:C_0805_2012Metric, F.Cu at (174.7, 84.0)
- added C4: 4.7uf, Capacitor_SMD:C_0805_2012Metric, F.Cu at (180.1, 79.5)
- added C5: 4.7uf, Capacitor_SMD:C_0805_2012Metric, F.Cu at (180.5, 76.2)
- added C6: 1uf, Capacitor_SMD:C_0805_2012Metric, F.Cu at (190.7, 71.7)
- added C7: 1uf, Capacitor_SMD:C_0805_2012Metric, F.Cu at (186.2, 71.7)
- added C8: 100nf, Capacitor_SMD:C_0805_2012Metric, F.Cu at (169.6, 86.2)
- added D44: D_Small, Diode_SMD:D_SOD-123, F.Cu at (170.2, 75.3)
- added D45: D_Small, Diode_SMD:D_SOD-123, F.Cu at (175.9, 71.9)
- added D46: D_Small, Diode_SMD:D_SOD-123, F.Cu at (170.2, 71.9)
- added F1: Polyfuse_Small, Fuse:Fuse_1206_3216Metric, F.Cu at (170.1, 78.6)
- added JP1: THERM, Jumper:SolderJumper-2_P1.3mm_Open_TrianglePad1.0x1.5mm, F.Cu at (198.2, 75.0)
- added L1: L, Capacitor_SMD:C_0402_1005Metric, F.Cu at (198.7, 71.2)
- added R1: 2.7k, Resistor_SMD:R_0805_2012Metric, F.Cu at (195.1, 71.7)
- added R10: 806k, Resistor_SMD:R_0805_2012Metric, F.Cu at (182.8, 86.9)
- added R11: 2M, Resistor_SMD:R_0805_2012Metric, F.Cu at (188.9, 80.6)
- added R2: 2.7k, Resistor_SMD:R_0805_2012Metric, F.Cu at (189.4, 77.7)
- added R3: 1.8k, Resistor_SMD:R_0805_2012Metric, F.Cu at (184.5, 82.1)
- added R4: 3.3k, Resistor_SMD:R_0805_2012Metric, F.Cu at (184.5, 79.2)
- added R5: 22k, Resistor_SMD:R_0805_2012Metric, F.Cu at (193.8, 74.7)
- added R6: 5.1k, Resistor_SMD:R_0805_2012Metric, F.Cu at (178.4, 87.0)
- added R7: 5.1k, Resistor_SMD:R_0805_2012Metric, F.Cu at (189.4, 74.7)
- added R8: 100, Resistor_SMD:R_0805_2012Metric, F.Cu at (179.1, 84.0)
- added R9: 1k, Resistor_SMD:R_0805_2012Metric, F.Cu at (193.8, 77.7)
- added U3: DW01A, Package_TO_SOT_SMD:SOT-23-6, F.Cu at (181.4, 72.5)
- added U4: FS8205, Package_TO_SOT_SMD:SOT-23-6, F.Cu at (169.9, 82.5)
- added U5: SRV05-4, marbastlib-various:SOT-23-6-routable, F.Cu at (175.7, 75.8)
- added U6: XC6206PxxxMR, Package_TO_SOT_SMD:SOT-23, F.Cu at (175.4, 80.3)
- D38, D39: value D_Small -> LED
- D43: value D_Small -> D_TVS
- J1: value Conn_01x04_Female -> Conn_01x04_Male
- SW1: value RotaryEncoder_Switch -> SW_Push
- U1: value E73-2G4M08S1C -> nRF52840_holyiot_18010
- U2: value MCP73831-2-OT -> TP4056
Connections:
- D10 pad 1: row_5 -> row_2
- D11 pad 1: row_4 -> row_1
- D12 pad 1: row_3 -> row_0
- D13 pad 1: row_2 -> row_5
- D14 pad 1: row_1 -> row_4
- D15 pad 1: row_0 -> row_3
- D16 pad 1: row_0 -> row_2
- D17 pad 1: row_5 -> row_1
- D18 pad 1: row_4 -> row_0
- D19 pad 1: row_3 -> row_5
- D20 pad 1: row_2 -> row_4
- D21 pad 1: row_1 -> row_3
- D22 pad 1: row_0 -> row_2
- D23 pad 1: row_5 -> row_1
- D24 pad 1: row_4 -> row_0
- D25 pad 1: row_3 -> row_5
- D26 pad 1: row_2 -> row_4
- D27 pad 1: row_1 -> row_3
- D28 pad 1: row_0 -> row_2
- D29 pad 1: row_5 -> row_1
- D30 pad 1: row_4 -> row_0
- D31 pad 1: row_3 -> row_5
- D32 pad 1: row_2 -> row_4
- D33 pad 1: row_1 -> row_3
- D34 pad 1: row_0 -> row_2
- D35 pad 1: row_4 -> row_1
- D36 pad 1: row_3 -> row_0
- D38 pad 1: row_4 -> Net-(D38-Pad1)
- D38 pad 2: Net-(D38-Pad2) -> +5V
- D39 pad 1: row_3 -> Net-(D39-Pad1)
- D39 pad 2: Net-(D39-Pad2) -> +5V
- D40 pad 1: row_2 -> row_0
- D42 pad 1: row_0 -> row_2
- D43 pad 1: row_5 -> GNDPWR
- D43 pad 2: Net-(D43-Pad2) -> GND
- D7 pad 1: row_0 -> row_5
- D7 pad 2: Net-(D35-Pad2) -> Net-(D7-Pad2)
- D8 pad 1: row_1 -> row_4
- D9 pad 1: row_2 -> row_3
- J1 pad 2: circle_Y -> vbus
- J1 pad 3: +5V -> scl
- J1 pad 4: circle_X -> sda
- J2 pad A6: d+ -> D+
- J2 pad A7: d- -> D-
- J2 pad B4: vbus -> VBUS
- J2 pad B6: d+ -> D+
- J2 pad B7: d- -> D-
- MX10 pad 2: Net-(D13-Pad2) -> Net-(D10-Pad2)
- MX11 pad 2: Net-(D14-Pad2) -> Net-(D11-Pad2)
- MX12 pad 2: Net-(D15-Pad2) -> Net-(D12-Pad2)
- MX13 pad 2: Net-(D17-Pad2) -> Net-(D13-Pad2)
- MX14 pad 2: Net-(D18-Pad2) -> Net-(D14-Pad2)
- MX15 pad 2: Net-(D19-Pad2) -> Net-(D15-Pad2)
- MX16 pad 2: Net-(D20-Pad2) -> Net-(D16-Pad2)
- MX17 pad 2: Net-(D21-Pad2) -> Net-(D17-Pad2)
- MX18 pad 2: Net-(D22-Pad2) -> Net-(D18-Pad2)
- MX19 pad 2: Net-(D23-Pad2) -> Net-(D19-Pad2)
- MX20 pad 2: Net-(D24-Pad2) -> Net-(D20-Pad2)
- MX21 pad 2: Net-(D25-Pad2) -> Net-(D21-Pad2)
- MX22 pad 2: Net-(D26-Pad2) -> Net-(D22-Pad2)
- MX23 pad 2: Net-(D27-Pad2) -> Net-(D23-Pad2)
- MX24 pad 2: Net-(D28-Pad2) -> Net-(D24-Pad2)
- MX25 pad 2: Net-(D29-Pad2) -> Net-(D25-Pad2)
- MX26 pad 2: Net-(D30-Pad2) -> Net-(D26-Pad2)
- MX27 pad 2: Net-(D31-Pad2) -> Net-(D27-Pad2)
- MX28 pad 2: Net-(D32-Pad2) -> Net-(D28-Pad2)
- MX29 pad 2: Net-(D33-Pad2) -> Net-(D29-Pad2)
- MX30 pad 2: Net-(D34-Pad2) -> Net-(D30-Pad2)
- MX31 pad 2: Net-(D37-Pad2) -> Net-(D31-Pad2)
- MX32 pad 2: Net-(D38-Pad2) -> Net-(D32-Pad2)
- MX33 pad 2: Net-(D39-Pad2) -> Net-(D33-Pad2)
- MX34 pad 2: Net-(D40-Pad2) -> Net-(D34-Pad2)
- MX35 pad 2: Net-(D41-Pad2) -> Net-(D35-Pad2)
- MX36 pad 2: Net-(D42-Pad2) -> Net-(D36-Pad2)
- MX37 pad 2: Net-(D43-Pad2) -> Net-(D37-Pad2)
- MX7 pad 2: Net-(D10-Pad2) -> Net-(D7-Pad2)
- MX8 pad 2: Net-(D11-Pad2) -> Net-(D8-Pad2)
- MX9 pad 2: Net-(D12-Pad2) -> Net-(D9-Pad2)
- S1 pad 1: Net-(D35-Pad2) -> Net-(D40-Pad2)
- S1 pad 4: Net-(D8-Pad2) -> Net-(D41-Pad2)
- S1 pad 6: Net-(D9-Pad2) -> Net-(D42-Pad2)
- S1 pad 7: Net-(D35-Pad2) -> Net-(D45-Pad2)
- S1 pad 9: Net-(D36-Pad2) -> Net-(D46-Pad2)
- SW1 pad A: encoder_top_A -> (no net)
- SW1 pad B: encoder_top_B -> (no net)
- SW1 pad C: GND -> (no net)
- SW1 pad S1: col_7 -> (no net)
- SW1 pad S2: Net-(D16-Pad2) -> (no net)
- U1 pad 11: unconnected-(U1-Pad11) -> VSENSE
- U1 pad 14: unconnected-(U1-Pad14) -> +3.3V
- U1 pad 15: circle_Y -> unconnected-(U1-Pad15)
- U1 pad 18: circle_X -> unconnected-(U1-Pad18)
- U1 pad 19: vdd -> unconnected-(U1-Pad19)
- U1 pad 21: GND -> reset
- U1 pad 22: unconnected-(U1-Pad22) -> vbus
- U1 pad 23: vddh -> d-
- U1 pad 24: GND -> d+
- U1 pad 25: dcch -> unconnected-(U1-Pad25)
- U1 pad 26: Net-(SW2-Pad1) -> unconnected-(U1-Pad26)
- U1 pad 27: vbus -> unconnected-(U1-Pad27)
- U1 pad 29: d+ -> unconnected-(U1-Pad29)
- U1 pad 3: encoder_bottom_B -> unconnected-(U1-Pad3)
- U1 pad 30: sda -> unconnected-(U1-Pad30)
- U1 pad 31: d+ -> swdclk
- U1 pad 32: scl -> swdio
- U1 pad 37: swdio -> unconnected-(U1-Pad37)
- U1 pad 39: swdclk -> unconnected-(U1-Pad39)
- U1 pad 4: encoder_top_A -> unconnected-(U1-Pad4)
- U1 pad 5: GND -> unconnected-(U1-Pad5)
- U1 pad 7: encoder_bottom_A -> unconnected-(U1-Pad7)
- U1 pad 8: encoder_top_B -> unconnected-(U1-Pad8)
- U2 pad 1: unconnected-(U2-Pad1) -> Net-(JP1-Pad2)
- U2 pad 2: GND -> Net-(R3-Pad1)
- U2 pad 3: Net-(BT1-Pad1) -> GND
- U2 pad 4: vbus -> +5V
- U2 pad 5: Net-(R1-Pad1) -> BAT+

Commit message: diod
Parts:
- C1, C2, C3, C4, C5, C6, C7, C8, D1, D10, D11, D12, D13, D14, D15, D16, D17, D18, D19, D2, D20, D21, D22, D23, D24, D25, D26, D27, D28, D29, D3, D30, D31, D32, D33, D34, D35, D36, D37, D38, D39, D4, D40, D41, D42, D43, D44, D45, D46, D5, D6, D7, D8, D9, F1, J2, JP1, L1, R1, R10, R11, R2, R3, R4, R5, R6, R7, R8, R9, U1, U2, U3, U4, U5, U6: moved to B.Cu
- MX36: footprint MX:MXOnly-1U-Hotswap -> MX:MXOnly-2U-Hotswap
- moved D37 252.0 mm to (31.0, 30.0), turned to 90 degrees
- moved D42 247.2 mm to (30.0, 37.0), turned to 180 degrees
- moved D40 239.9 mm to (19.0, 53.0)
- moved S1 233.4 mm to (25.0, 45.0)
- moved D33 213.2 mm to (50.0, 68.0), turned to 90 degrees
- moved D41 211.1 mm to (36.0, 48.0), turned to 90 degrees
- moved D35 202.9 mm to (50.0, 106.0), turned to 90 degrees
- moved D32 199.7 mm to (50.0, 49.0), turned to 90 degrees
- moved D26 196.0 mm to (69.0, 49.0), turned to 90 degrees
- moved D25 193.0 mm to (69.0, 30.0), turned to 90 degrees
- moved D19 192.9 mm to (88.0, 30.0), turned to 90 degrees
- moved SW1 191.7 mm to (25.0, 112.0)
- moved D28 190.3 mm to (69.0, 87.0), turned to 90 degrees
- moved D36 187.9 mm to (38.0, 133.0), turned to 110 degrees
- moved D21 185.9 mm to (88.0, 68.0), turned to 90 degrees
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
Commit message: rows :)
Parts:
- moved D30 0.97 mm to (67.5, 125.8)
- moved D36 0.50 mm to (37.6, 133.3)
- turned D22 to 90 degrees
Routing:
- net Net-(D36-Pad2): track 0.00 -> 8.87 mm
- net Net-(D30-Pad2): track 0.00 -> 8.85 mm
- net Net-(D29-Pad2): track 0.00 -> 8.75 mm
- net Net-(D26-Pad2): track 0.00 -> 8.74 mm
- net Net-(D28-Pad2): track 0.00 -> 8.74 mm
- net Net-(D32-Pad2): track 0.00 -> 8.74 mm
- net Net-(D35-Pad2): track 0.00 -> 8.74 mm
- net Net-(D27-Pad2): track 0.00 -> 8.74 mm
- net Net-(D34-Pad2): track 0.00 -> 8.74 mm
- net Net-(D33-Pad2): track 0.00 -> 8.74 mm
- net Net-(D24-Pad2): track 0.00 -> 8.73 mm
- net Net-(D23-Pad2): track 0.00 -> 8.73 mm
- net Net-(D22-Pad2): track 0.00 -> 8.73 mm
- net Net-(D20-Pad2): track 0.00 -> 8.73 mm
- net Net-(D18-Pad2): track 0.00 -> 8.73 mm
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
Commit message: cols
Parts:
- moved D43 31.1 mm to (170.0, 59.0)
- moved L1 30.8 mm to (216.0, 68.0)
Routing:
- net row_5: track 0.00 -> 128.4 mm
- net row_2: track 0.00 -> 123.7 mm
- net row_1: track 0.00 -> 123.7 mm
- net row_4: track 0.00 -> 121.2 mm
- net row_3: track 0.00 -> 121.2 mm
- net row_0: track 0.00 -> 88.3 mm

Commit message: wicked cols
Parts:
- moved JP1 268.6 mm to (-75.6, 71.0)
- moved D44 260.1 mm to (-39.4, 105.6)
- moved U5 260.1 mm to (-44.9, 106.1)
- moved C2 260.1 mm to (-54.2, 106.5)
- moved C5 260.1 mm to (-49.7, 106.5)
- moved R2 260.1 mm to (-58.6, 108.0)
- moved R5 260.1 mm to (-63.0, 105.0)
- moved R7 260.1 mm to (-58.6, 105.0)
- moved R9 260.1 mm to (-63.0, 108.0)
- moved C8 257.6 mm to (-33.7, 141.3)
- moved R6 257.6 mm to (-42.6, 142.1)
- moved C1 257.6 mm to (-38.2, 142.1)
- moved R10 257.6 mm to (-47.0, 142.0)
- moved C6 256.0 mm to (-56.2, 85.1)
- moved C7 256.0 mm to (-51.7, 85.1)
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Routing:
- net col_5: track 0.00 -> 129.8 mm, vias 0 -> 6
- net col_4: track 0.00 -> 114.3 mm, vias 0 -> 6
- net col_1: track 0.00 -> 111.2 mm, vias 0 -> 6
- net col_0: track 0.00 -> 110.7 mm, vias 0 -> 6
- net col_2: track 0.00 -> 110.7 mm, vias 0 -> 6
- net col_3: track 0.00 -> 110.6 mm, vias 0 -> 6
- net row_4: track 121.2 -> 163.9 mm
- net col_6: track 0.00 -> 37.4 mm
- net row_1: track 123.7 -> 130.4 mm
- net row_2: track 123.7 -> 130.4 mm
- net row_5: track 128.4 -> 135.0 mm
- net row_3: track 121.2 -> 127.8 mm
- net Net-(D45-Pad2): track 0.00 -> 5.68 mm
- net Net-(D42-Pad2): track 0.00 -> 4.77 mm
- net Net-(D41-Pad2): track 0.00 -> 4.46 mm
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