File: kicad/left/alleycat_left.kicad_pcb (KiCad board)
At the start: 2 copper layers, 134 x 128 mm, 84 parts, among them J1 Conn_01x04_Female, SW1 RotaryEncoder_Switch, U1 E73-2G4M08S1C

Commit message: do it for the left side too
Parts:
- added U2: MCP73831-2-OT, Package_TO_SOT_SMD:SOT-23-5, F.Cu at (168.0, 136.0)
Connections:
- U1 pad 15: unconnected-(U1-Pad15) -> circle_Y
- U1 pad 18: unconnected-(U1-Pad18) -> circle_X
- U1 pad 19: unconnected-(U1-Pad19) -> vdd
- U1 pad 21: unconnected-(U1-Pad21) -> GND
- U1 pad 23: unconnected-(U1-Pad23) -> vddh
- U1 pad 24: unconnected-(U1-Pad24) -> GND
- U1 pad 25: unconnected-(U1-Pad25) -> dcch
- U1 pad 26: unconnected-(U1-Pad26) -> Net-(SW2-Pad1)
- U1 pad 27: unconnected-(U1-Pad27) -> vbus
- U1 pad 29: unconnected-(U1-Pad29) -> d+
- U1 pad 3: unconnected-(U1-Pad3) -> encoder_bottom_B
- U1 pad 30: unconnected-(U1-Pad30) -> sda
- U1 pad 31: unconnected-(U1-Pad31) -> d+
- U1 pad 32: unconnected-(U1-Pad32) -> scl
- U1 pad 37: unconnected-(U1-Pad37) -> swdio
- U1 pad 39: unconnected-(U1-Pad39) -> swdclk
- U1 pad 4: unconnected-(U1-Pad4) -> encoder_top_A
- U1 pad 5: unconnected-(U1-Pad5) -> GND
- U1 pad 7: unconnected-(U1-Pad7) -> encoder_bottom_A
- U1 pad 8: unconnected-(U1-Pad8) -> encoder_top_B

Commit message: ANY ALIGNERS?
Parts:
- MX1, MX10, MX11, MX12, MX13, MX14, MX15, MX16, MX17, MX18, MX19, MX2, MX20, MX21, MX22, MX23, MX24, MX25, MX26, MX27, MX28, MX29, MX3, MX30, MX31, MX32, MX33, MX34, MX35, MX36, MX37, MX4, MX5, MX6, MX7, MX8, MX9: value MX-NoLED -> 1U; footprint MX:MX-NoLED -> MX:MXOnly-1U-Hotswap
- moved MX11 341.4 mm to (37.0, 99.0)
- moved MX3 317.6 mm to (18.0, 61.0)
- moved MX29 289.1 mm to (94.0, 99.0)
- moved MX10 280.2 mm to (37.0, 80.0)
- moved MX9 280.1 mm to (37.0, 61.0)
- moved MX5 278.3 mm to (18.0, 99.0)
- moved MX18 272.0 mm to (56.0, 118.0)
- moved MX30 253.4 mm to (95.7, 118.1), turned to -10 degrees
- moved MX32 243.6 mm to (113.0, 42.0)
- moved MX27 243.4 mm to (94.0, 61.0)
- moved MX19 241.4 mm to (75.0, 23.0)
- moved MX16 240.1 mm to (56.0, 80.0)
- moved MX4 238.7 mm to (18.0, 80.0)
- moved MX12 225.7 mm to (37.0, 118.0)
- moved MX7 221.2 mm to (36.9, 23.0)
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
Commit message: uhh uhhh uhhh uhh uhhh uhhh uhhh uuhhh uhhh uhh uhh uhhhu hh uhh footprints
Parts:
- added C1: 10uf, Capacitor_SMD:C_0805_2012Metric, F.Cu at (200.0, 86.0)
- added C2: 100nf, Capacitor_SMD:C_0805_2012Metric, F.Cu at (189.9, 93.5)
- added C3: 100nf, Capacitor_SMD:C_0805_2012Metric, F.Cu at (179.2, 102.7)
- added C4: 4.7uf, Capacitor_SMD:C_0805_2012Metric, F.Cu at (185.5, 96.8)
- added C5: 4.7uf, Capacitor_SMD:C_0805_2012Metric, F.Cu at (185.5, 93.8)
- added C6: 1uf, Capacitor_SMD:C_0805_2012Metric, F.Cu at (194.3, 90.5)
- added C7: 1uf, Capacitor_SMD:C_0805_2012Metric, F.Cu at (195.6, 86.0)
- added C8: 100nf, Capacitor_SMD:C_0805_2012Metric, F.Cu at (189.9, 90.5)
- added D44: D_Small, Diode_SMD:D_SOD-123, F.Cu at (185.3, 86.2)
- added D45: D_Small, Diode_SMD:D_SOD-123, F.Cu at (174.8, 98.5)
- added D46: D_Small, Diode_SMD:D_SOD-123, F.Cu at (174.8, 95.2)
- added F1: Polyfuse_Small, Fuse:Fuse_1206_3216Metric, F.Cu at (180.4, 95.1)
- added J2: USB_C_Receptacle_USB2.0, MX:TYPE-C-31-M-12, F.Cu at (177.2, 85.6)
- added JP1: THERM, Jumper:SolderJumper-2_P1.3mm_Open_TrianglePad1.0x1.5mm, F.Cu at (193.5, 99.7)
- added L1: L, Capacitor_SMD:C_0402_1005Metric, F.Cu at (198.0, 94.4)
- added R1: 2.7k, Resistor_SMD:R_0805_2012Metric, F.Cu at (198.8, 89.0)
- added R10: 806k, Resistor_SMD:R_0805_2012Metric, F.Cu at (198.8, 91.9)
- added R11: 2M, Resistor_SMD:R_0805_2012Metric, F.Cu at (188.1, 102.7)
- added R2: 2.7k, Resistor_SMD:R_0805_2012Metric, F.Cu at (204.4, 86.0)
- added R3: 1.8k, Resistor_SMD:R_0805_2012Metric, F.Cu at (189.1, 99.8)
- added R4: 3.3k, Resistor_SMD:R_0805_2012Metric, F.Cu at (189.9, 96.4)
- added R5: 22k, Resistor_SMD:R_0805_2012Metric, F.Cu at (194.3, 96.4)
- added R6: 5.1k, Resistor_SMD:R_0805_2012Metric, F.Cu at (183.7, 102.7)
- added R7: 5.1k, Resistor_SMD:R_0805_2012Metric, F.Cu at (194.3, 93.4)
- added R8: 100, Resistor_SMD:R_0805_2012Metric, F.Cu at (184.7, 99.8)
- added R9: 1k, Resistor_SMD:R_0805_2012Metric, F.Cu at (203.2, 89.0)
- added U3: DW01A, Package_TO_SOT_SMD:SOT-23-6, F.Cu at (190.8, 86.7)
- added U4: FS8205, Package_TO_SOT_SMD:SOT-23-6, F.Cu at (174.4, 102.4)
- added U5: SRV05-4, marbastlib-various:SOT-23-6-routable, F.Cu at (185.1, 90.1)
- added U6: XC6206PxxxMR, Package_TO_SOT_SMD:SOT-23, F.Cu at (180.1, 99.0)
- D38, D39: value D_Small -> LED
- D43: value D_Small -> D_TVS
- J1: value Conn_01x04_Female -> Conn_01x04_Male
- MX1, MX10, MX11, MX12, MX13, MX14, MX15, MX16, MX17, MX18, MX19, MX2, MX20, MX21, MX22, MX23, MX24, MX25, MX26, MX27, MX28, MX29, MX3, MX30, MX31, MX32, MX33, MX34, MX35, MX36, MX37, MX4, MX5, MX6, MX7, MX8, MX9: value 1U -> MX-NoLED
- SW1: value RotaryEncoder_Switch -> SW_Push
- U1: value E73-2G4M08S1C -> nRF52840_holyiot_18010
- U2: value MCP73831-2-OT -> TP4056
Connections:
- net vddh renamed d-
- D10 pad 1: row_5 -> row_2
- D11 pad 1: row_4 -> row_1
- D12 pad 1: row_3 -> row_0
- D13 pad 1: row_2 -> row_5
- D14 pad 1: row_1 -> row_4
- D15 pad 1: row_0 -> row_3
- D16 pad 1: row_0 -> row_2
- D17 pad 1: row_5 -> row_1
- D18 pad 1: row_4 -> row_0
- D19 pad 1: row_3 -> row_5
- D20 pad 1: row_2 -> row_4
- D21 pad 1: row_1 -> row_3
- D22 pad 1: row_0 -> row_2
- D23 pad 1: row_5 -> row_1
- D24 pad 1: row_4 -> row_0
- D25 pad 1: row_3 -> row_5
- D26 pad 1: row_2 -> row_4
- D27 pad 1: row_1 -> row_3
- D28 pad 1: row_0 -> row_2
- D29 pad 1: row_5 -> row_1
- D30 pad 1: row_4 -> row_0
- D31 pad 1: row_3 -> row_5
- D32 pad 1: row_2 -> row_4
- D33 pad 1: row_1 -> row_3
- D34 pad 1: row_0 -> row_2
- D35 pad 1: row_4 -> row_1
- D36 pad 1: row_3 -> row_0
- D38 pad 1: row_4 -> Net-(D38-Pad1)
- D38 pad 2: Net-(D38-Pad2) -> +5V
- D39 pad 1: row_3 -> Net-(D39-Pad1)
- D39 pad 2: Net-(D39-Pad2) -> +5V
- D40 pad 1: row_2 -> row_0
- D42 pad 1: row_0 -> row_2
- D43 pad 1: row_5 -> GNDPWR
- D43 pad 2: Net-(D43-Pad2) -> GND
- D7 pad 1: row_0 -> row_5
- D7 pad 2: Net-(D35-Pad2) -> Net-(D7-Pad2)
- D8 pad 1: row_1 -> row_4
- D9 pad 1: row_2 -> row_3
- J1 pad 2: circle_Y -> vbus
- J1 pad 3: +5V -> scl
- J1 pad 4: circle_X -> sda
- MX10 pad 2: Net-(D13-Pad2) -> Net-(D10-Pad2)
- MX11 pad 2: Net-(D14-Pad2) -> Net-(D11-Pad2)
- MX12 pad 2: Net-(D15-Pad2) -> Net-(D12-Pad2)
- MX13 pad 2: Net-(D17-Pad2) -> Net-(D13-Pad2)
- MX14 pad 2: Net-(D18-Pad2) -> Net-(D14-Pad2)
- MX15 pad 2: Net-(D19-Pad2) -> Net-(D15-Pad2)
- MX16 pad 2: Net-(D20-Pad2) -> Net-(D16-Pad2)
- MX17 pad 2: Net-(D21-Pad2) -> Net-(D17-Pad2)
- MX18 pad 2: Net-(D22-Pad2) -> Net-(D18-Pad2)
- MX19 pad 2: Net-(D23-Pad2) -> Net-(D19-Pad2)
- MX20 pad 2: Net-(D24-Pad2) -> Net-(D20-Pad2)
- MX21 pad 2: Net-(D25-Pad2) -> Net-(D21-Pad2)
- MX22 pad 2: Net-(D26-Pad2) -> Net-(D22-Pad2)
- MX23 pad 2: Net-(D27-Pad2) -> Net-(D23-Pad2)
- MX24 pad 2: Net-(D28-Pad2) -> Net-(D24-Pad2)
- MX25 pad 2: Net-(D29-Pad2) -> Net-(D25-Pad2)
- MX26 pad 2: Net-(D30-Pad2) -> Net-(D26-Pad2)
- MX27 pad 2: Net-(D31-Pad2) -> Net-(D27-Pad2)
- MX28 pad 2: Net-(D32-Pad2) -> Net-(D28-Pad2)
- MX29 pad 2: Net-(D33-Pad2) -> Net-(D29-Pad2)
- MX30 pad 2: Net-(D34-Pad2) -> Net-(D30-Pad2)
- MX31 pad 2: Net-(D37-Pad2) -> Net-(D31-Pad2)
- MX32 pad 2: Net-(D38-Pad2) -> Net-(D32-Pad2)
- MX33 pad 2: Net-(D39-Pad2) -> Net-(D33-Pad2)
- MX34 pad 2: Net-(D40-Pad2) -> Net-(D34-Pad2)
- MX35 pad 2: Net-(D41-Pad2) -> Net-(D35-Pad2)
- MX36 pad 2: Net-(D42-Pad2) -> Net-(D36-Pad2)
- MX37 pad 2: Net-(D43-Pad2) -> Net-(D37-Pad2)
- MX7 pad 2: Net-(D10-Pad2) -> Net-(D7-Pad2)
- MX8 pad 2: Net-(D11-Pad2) -> Net-(D8-Pad2)
- MX9 pad 2: Net-(D12-Pad2) -> Net-(D9-Pad2)
- S1 pad 1: Net-(D35-Pad2) -> Net-(D40-Pad2)
- S1 pad 4: Net-(D8-Pad2) -> Net-(D41-Pad2)
- S1 pad 6: Net-(D9-Pad2) -> Net-(D42-Pad2)
- S1 pad 7: Net-(D35-Pad2) -> Net-(D45-Pad2)
- S1 pad 9: Net-(D36-Pad2) -> Net-(D46-Pad2)
- SW1 pad A: encoder_top_A -> (no net)
- SW1 pad B: encoder_top_B -> (no net)
- SW1 pad C: GND -> (no net)
- SW1 pad S1: col_7 -> (no net)
- SW1 pad S2: Net-(D16-Pad2) -> (no net)
- U1 pad 11: unconnected-(U1-Pad11) -> VSENSE
- U1 pad 14: unconnected-(U1-Pad14) -> +3.3V
- U1 pad 15: circle_Y -> unconnected-(U1-Pad15)
- U1 pad 18: circle_X -> unconnected-(U1-Pad18)
- U1 pad 19: vdd -> unconnected-(U1-Pad19)
- U1 pad 21: GND -> reset
- U1 pad 22: unconnected-(U1-Pad22) -> vbus
- U1 pad 24: GND -> d+
- U1 pad 25: dcch -> unconnected-(U1-Pad25)
- U1 pad 26: Net-(SW2-Pad1) -> unconnected-(U1-Pad26)
- U1 pad 27: vbus -> unconnected-(U1-Pad27)
- U1 pad 29: d+ -> unconnected-(U1-Pad29)
- U1 pad 3: encoder_bottom_B -> unconnected-(U1-Pad3)
- U1 pad 30: sda -> unconnected-(U1-Pad30)
- U1 pad 31: d+ -> swdclk
- U1 pad 32: scl -> swdio
- U1 pad 37: swdio -> unconnected-(U1-Pad37)
- U1 pad 39: swdclk -> unconnected-(U1-Pad39)
- U1 pad 4: encoder_top_A -> unconnected-(U1-Pad4)
- U1 pad 5: GND -> unconnected-(U1-Pad5)
- U1 pad 7: encoder_bottom_A -> unconnected-(U1-Pad7)
- U1 pad 8: encoder_top_B -> unconnected-(U1-Pad8)
- U2 pad 1: unconnected-(U2-Pad1) -> Net-(JP1-Pad2)
- U2 pad 2: GND -> Net-(R3-Pad1)
- U2 pad 3: Net-(BT1-Pad1) -> GND
- U2 pad 4: vbus -> +5V
- U2 pad 5: Net-(R1-Pad1) -> BAT+

Commit message: nyaaaa
Parts:
- added SW2: RotaryEncoder_Switch, Keebio-Parts:RotaryEncoder_Alps_EC11E-Switch_Vertical_H20mm, F.Cu at (139.5, 43.0)
- D1, D10, D11, D12, D13, D14, D15, D16, D17, D18, D19, D2, D20, D21, D22, D23, D24, D25, D26, D27, D28, D29, D3, D30, D31, D32, D33, D34, D35, D36, D37, D4, D40, D41, D42, D5, D6, D7, D8, D9, U1: moved to B.Cu
- D38, D39: footprint Diode_SMD:D_SOD-123 -> LED_SMD:LED_0805_2012Metric
- D43: footprint Diode_SMD:D_SOD-123 -> MX:SOD-323; moved to B.Cu
- MX36: footprint MX:MXOnly-1U-Hotswap -> MX:MXOnly-2U-Hotswap
- SW1: footprint Keebio-Parts:RotaryEncoder_Alps_EC11E-Switch_Vertical_H20mm -> Keebio-Parts:SW_SPST_TL3342
- U2: footprint Package_TO_SOT_SMD:SOT-23-5 -> Package_SO:SOP-8-1EP_4.57x4.57mm_P1.27mm_EP4.57x4.45mm
- moved D1 287.2 mm to (-2.00, 14.0), turned to 90 degrees
- moved D7 261.8 mm to (5.00, 26.0), turned to 90 degrees
- moved D5 223.7 mm to (31.0, 106.0), turned to 90 degrees
- moved D8 217.7 mm to (50.0, 49.0), turned to 90 degrees
- moved D14 205.3 mm to (69.0, 49.0), turned to 90 degrees
- moved D6 202.0 mm to (31.0, 125.0), turned to 90 degrees
- moved D4 200.9 mm to (31.0, 87.0), turned to 90 degrees
- moved D43 199.6 mm to (16.0, 14.0)
- moved D9 199.6 mm to (50.0, 68.0), turned to 90 degrees
- moved D17 196.0 mm to (69.0, 106.0), turned to 90 degrees
- moved D13 195.6 mm to (69.0, 30.0), turned to 90 degrees
- moved D10 195.0 mm to (50.0, 87.0), turned to 90 degrees
- moved D19 192.9 mm to (88.0, 30.0), turned to 90 degrees
- moved D21 185.9 mm to (88.0, 68.0), turned to 90 degrees
- moved D11 182.6 mm to (50.0, 106.0), turned to 90 degrees
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Routing:
- net col_5: track 0.00 -> 106.2 mm
- net col_4: track 0.00 -> 95.8 mm
- net col_2: track 0.00 -> 95.0 mm
- net col_3: track 0.00 -> 95.0 mm
- net col_1: track 0.00 -> 76.2 mm
- net col_0: track 0.00 -> 76.0 mm

Commit message: did a little pcbing
Parts:
- C1, C2, C3, C4, C5, C6, C7, C8, D38, D39, D44, D45, D46, F1, JP1, L1, R1, R10, R11, R2, R3, R4, R5, R6, R7, R8, R9, U2, U3, U4, U5, U6: moved to B.Cu
- moved F1 192.8 mm to (10.0, 5.00), turned to 180 degrees
- moved R1 67.0 mm to (132.0, 95.0), turned to -90 degrees
- moved R2 58.1 mm to (147.0, 95.0), turned to -90 degrees
- moved D44 57.6 mm to (144.0, 46.0), turned to 90 degrees
- moved U2 46.2 mm to (182.0, 92.0), turned to 180 degrees
- moved D46 42.5 mm to (133.0, 103.0), turned to -140 degrees
- moved U5 40.6 mm to (222.4, 74.1), turned to 180 degrees
- moved D45 40.5 mm to (135.0, 106.0), turned to 90 degrees
- moved C4 39.9 mm to (222.1, 80.8), turned to 180 degrees
- moved C5 39.9 mm to (222.1, 77.8), turned to 180 degrees
- moved D1 37.6 mm to (34.0, 3.00)
- moved C8 32.0 mm to (217.6, 74.5), turned to 180 degrees
- moved R10 29.0 mm to (170.0, 88.0), turned to 180 degrees
- moved C1 28.7 mm to (175.0, 100.0), turned to 180 degrees
- moved R11 27.6 mm to (213.1, 91.0), turned to 180 degrees
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
Commit message: pcb edit pog pog pog
Parts:
- U1: footprint E73-2G4M08S1C:E73-2G4M08S1C -> marbastlib-various:nRF52840_holyiot_18010
- U2: footprint Package_SO:SOP-8-1EP_4.57x4.57mm_P1.27mm_EP4.57x4.45mm -> Package_TO_SOT_SMD:SOT-23-5
- moved U5 53.4 mm to (169.0, 73.0)
- moved U4 52.8 mm to (133.0, 98.0), turned to 0 degrees
- moved U2 48.1 mm to (136.0, 78.0)
- moved D7 38.9 mm to (50.0, 30.0)
- moved D39 30.5 mm to (169.0, 82.0)
- moved R1 29.7 mm to (157.0, 79.0)
- moved R2 29.7 mm to (172.0, 79.0)
- moved D38 28.8 mm to (160.0, 82.0)
- moved D1 27.2 mm to (31.0, 30.0)
- moved U3 13.5 mm to (162.0, 73.0)
- moved D43 10.0 mm to (16.0, 5.00)
- moved D45 10.0 mm to (145.0, 106.0)
- moved J1 3.00 mm to (145.5, 54.1)
- moved SW1 1.00 mm to (139.6, 84.0)
- turned D36 to 70 degrees
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Connections:
- J1 pad 2: vbus -> +5V
Routing:
- net row_3: track 0.00 -> 118.3 mm
- net row_2: track 0.00 -> 108.3 mm
- net row_1: track 0.00 -> 107.2 mm
- net row_5: track 0.00 -> 94.5 mm
- net row_0: track 0.00 -> 76.1 mm
- net row_4: track 0.00 -> 66.3 mm
- net col_1: track 76.2 -> 95.8 mm, vias 0 -> 6
- net col_0: track 76.0 -> 95.0 mm
- net col_4: track 95.8 -> 112.5 mm, vias 0 -> 6
- net col_3: track 95.0 -> 111.3 mm, vias 0 -> 6
- net col_2: track 95.0 -> 111.3 mm, vias 0 -> 6
- net col_5: track 106.2 -> 122.5 mm, vias 0 -> 6
- net Net-(D3-Pad2): track 0.00 -> 8.90 mm
- net Net-(D18-Pad2): track 0.00 -> 8.75 mm
- net Net-(D30-Pad2): track 0.00 -> 8.74 mm
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
Commit message: pogged
Parts:
- U2: footprint Package_TO_SOT_SMD:SOT-23-5 -> Package_SO:SOP-8-1EP_4.57x4.57mm_P1.27mm_EP4.57x4.45mm
- moved J1 5.77 mm to (147.8, 59.4)
- moved MX37 3.91 mm to (134.5, 20.0)
- moved S1 3.50 mm to (142.8, 112.1)
- moved MX1 3.00 mm to (18.0, 20.0)
- moved MX13 3.00 mm to (56.0, 20.0)
- moved MX19 3.00 mm to (75.0, 20.0)
- moved MX25 3.00 mm to (94.0, 20.0)
- moved MX31 3.00 mm to (113.0, 20.0)
- moved MX7 3.00 mm to (36.9, 20.0)
- moved SW2 2.90 mm to (141.5, 45.1)
- moved MX36 1.39 mm to (125.2, 125.6)
- moved D30 0.47 mm to (107.4, 127.2)
- moved MX30 0.47 mm to (96.1, 118.3)
Other:
- board size 134 x 128 mm -> 139.8 x 136.9 mm
