File: kicad/left/alleycat_left.kicad_pcb (KiCad board)
At the start: 2 copper layers, 139.8 x 136.9 mm, 116 parts, among them J1 Conn_01x04_Male, J2 USB_C_Receptacle_USB2.0, SW1 SW_Push, SW2 RotaryEncoder_Switch, U1 nRF52840_holyiot_18010, U2 TP4056, U3 DW01A, U4 FS8205, U5 SRV05-4, U6 XC6206PxxxMR

Commit message: nya
Parts:
- moved U2 6.50 mm to (142.2, 80.1)
- moved SW1 4.66 mm to (142.0, 88.0)
- moved MX36 0.12 mm to (125.3, 125.7)
